File: hardware/pcb/dumta.kicad_sch (KiCad schematic)
At the start: 41 parts, among them J2 nice_view, SW1 SW_PUSH, SW10 SW_PUSH, SW11 SW_PUSH, SW12 SW_PUSH, SW13 SW_PUSH, SW14 SW_PUSH, SW15 SW_PUSH, SW16 SW_PUSH, SW17 SW_PUSH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

Commit message: feat: change footprints and alter them to match design rules
Parts:
- BT1: footprint swoop:Battery_pads_reversible -> dumta:Battery_pads_reversible
- D1, D10, D11, D12, D13, D14, D15, D16, D17, D18, D2, D3, D4, D5, D6, D7, D8, D9: footprint swoop:D_SMD_TH -> dumta:D_SMD_TH
- SW1, SW10, SW11, SW12, SW13, SW14, SW15, SW16, SW17, SW18, SW2, SW3, SW4, SW5, SW6, SW7, SW8, SW9: footprint keyswitches:Kailh_socket_PG1350_reversible -> dumta:Kailh_socket_PG1350_reversible
- U1: footprint swoop:ProMicro_jumpers -> dumta:ProMicro_jumpers
Changed lines of the file:
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@@
       (effects (font (size 1.524 1.524)))
     )
-    (property "Footprint" "swoop:ProMicro_jumpers" (at 170.18 71.12 0)
+    (property "Footprint" "dumta:ProMicro_jumpers" (at 170.18 71.12 0)
       (effects (font (size 1.524 1.524)) hide)
     )
@@
       (effects (font (size 1.27 1.27)))
     )
-    (property "Footprint" "keyswitches:Kailh_socket_PG1350_reversible" (at 49.53 43.815 0)
+    (property "Footprint" "dumta:Kailh_socket_PG1350_reversible" (at 49.53 43.815 0)
       (effects (font (size 1.27 1.27)) hide)
     )
@@
       (effects (font (size 1.27 1.27)))
     )
-    (property "Footprint" "swoop:D_SMD_TH" (at 57.15 47.625 0)
+    (property "Footprint" "dumta:D_SMD_TH" (at 57.15 47.625 0)
       (effects (font (size 1.27 1.27)) hide)
     )
@@
       (effects (font (size 1.27 1.27)))
     )
-    (property "Footprint" "keyswitches:Kailh_socket_PG1350_reversible" (at 67.31 43.815 0)
+    (property "Footprint" "dumta:Kailh_socket_PG1350_reversible" (at 67.31 43.815 0)
       (effects (font (size 1.27 1.27)) hide)
     )
@@
       (effects (font (size 1.27 1.27)))
     )
-    (property "Footprint" "swoop:D_SMD_TH" (at 74.93 47.625 0)
+    (property "Footprint" "dumta:D_SMD_TH" (at 74.93 47.625 0)
       (effects (font (size 1.27 1.27)) hide)
     )
@@
       (effects (font (size 1.27 1.27)))
     )
-    (property "Footprint" "keyswitches:Kailh_socket_PG1350_reversible" (at 85.09 43.815 0)
+    (property "Footprint" "dumta:Kailh_socket_PG1350_reversible" (at 85.09 43.815 0)
       (effects (font (size 1.27 1.27)) hide)
     )
@@
       (effects (font (size 1.27 1.27)))
     )
-    (property "Footprint" "keyswitches:Kailh_socket_PG1350_reversible" (at 102.87 43.815 0)
+    (property "Footprint" "dumta:Kailh_socket_PG1350_reversible" (at 102.87 43.815 0)
       (effects (font (size 1.27 1.27)) hide)
     )
@@
       (effects (font (size 1.27 1.27)))
     )
-    (property "Footprint" "keyswitches:Kailh_socket_PG1350_reversible" (at 120.65 43.815 0)
+    (property "Footprint" "dumta:Kailh_socket_PG1350_reversible" (at 120.65 43.815 0)
       (effects (font (size 1.27 1.27)) hide)
     )
@@
       (effects (font (size 1.27 1.27)))
     )
-    (property "Footprint" "swoop:D_SMD_TH" (at 92.71 47.625 0)
+    (property "Footprint" "dumta:D_SMD_TH" (at 92.71 47.625 0)
       (effects (font (size 1.27 1.27)) hide)
     )
@@
       (effects (font (size 1.27 1.27)))
     )
-    (property "Footprint" "swoop:D_SMD_TH" (at 110.49 47.625 0)
+    (property "Footprint" "dumta:D_SMD_TH" (at 110.49 47.625 0)
       (effects (font (size 1.27 1.27)) hide)
     )
@@
       (effects (font (size 1.27 1.27)))
     )
-    (property "Footprint" "swoop:D_SMD_TH" (at 128.27 47.625 0)
+    (property "Footprint" "dumta:D_SMD_TH" (at 128.27 47.625 0)
       (effects (font (size 1.27 1.27)) hide)
     )
@@
       (effects (font (size 1.27 1.27)))
     )
-    (property "Footprint" "keyswitches:Kailh_socket_PG1350_reversible" (at 49.53 59.055 0)
+    (property "Footprint" "dumta:Kailh_socket_PG1350_reversible" (at 49.53 59.055 0)
       (effects (font (size 1.27 1.27)) hide)
     )
@@
       (effects (font (size 1.27 1.27)))
     )
-    (property "Footprint" "swoop:D_SMD_TH" (at 57.15 62.865 0)
+    (property "Footprint" "dumta:D_SMD_TH" (at 57.15 62.865 0)
       (effects (font (size 1.27 1.27)) hide)
     )
@@
       (effects (font (size 1.27 1.27)))
     )
-    (property "Footprint" "keyswitches:Kailh_socket_PG1350_reversible" (at 67.31 59.055 0)
+    (property "Footprint" "dumta:Kailh_socket_PG1350_reversible" (at 67.31 59.055 0)
       (effects (font (size 1.27 1.27)) hide)
     )
@@
       (effects (font (size 1.27 1.27)))
     )
-    (property "Footprint" "swoop:D_SMD_TH" (at 74.93 62.865 0)
+    (property "Footprint" "dumta:D_SMD_TH" (at 74.93 62.865 0)
       (effects (font (size 1.27 1.27)) hide)
     )
@@
       (effects (font (size 1.27 1.27)))
     )
-    (property "Footprint" "keyswitches:Kailh_socket_PG1350_reversible" (at 85.09 59.055 0)
+    (property "Footprint" "dumta:Kailh_socket_PG1350_reversible" (at 85.09 59.055 0)
       (effects (font (size 1.27 1.27)) hide)
     )
@@
       (effects (font (size 1.27 1.27)))
     )
-    (property "Footprint" "keyswitches:Kailh_socket_PG1350_reversible" (at 102.87 59.055 0)
+    (property "Footprint" "dumta:Kailh_socket_PG1350_reversible" (at 102.87 59.055 0)
       (effects (font (size 1.27 1.27)) hide)
     )
@@
       (effects (font (size 1.27 1.27)))
     )
-    (property "Footprint" "keyswitches:Kailh_socket_PG1350_reversible" (at 120.65 59.055 0)
+    (property "Footprint" "dumta:Kailh_socket_PG1350_reversible" (at 120.65 59.055 0)
       (effects (font (size 1.27 1.27)) hide)
     )
@@
       (effects (font (size 1.27 1.27)))
     )
-    (property "Footprint" "swoop:D_SMD_TH" (at 92.71 62.865 0)
+    (property "Footprint" "dumta:D_SMD_TH" (at 92.71 62.865 0)
       (effects (font (size 1.27 1.27)) hide)
     )
@@
       (effects (font (size 1.27 1.27)))
     )
-    (property "Footprint" "swoop:D_SMD_TH" (at 110.49 62.865 0)
+    (property "Footprint" "dumta:D_SMD_TH" (at 110.49 62.865 0)
       (effects (font (size 1.27 1.27)) hide)
     )
@@
       (effects (font (size 1.27 1.27)))
     )
-    (property "Footprint" "swoop:D_SMD_TH" (at 128.27 62.865 0)
+    (property "Footprint" "dumta:D_SMD_TH" (at 128.27 62.865 0)
       (effects (font (size 1.27 1.27)) hide)
     )
@@
       (effects (font (size 1.27 1.27)))
     )
-    (property "Footprint" "keyswitches:Kailh_socket_PG1350_reversible" (at 49.53 74.295 0)
+    (property "Footprint" "dumta:Kailh_socket_PG1350_reversible" (at 49.53 74.295 0)
       (effects (font (size 1.27 1.27)) hide)
     )
@@
       (effects (font (size 1.27 1.27)))
     )
-    (property "Footprint" "swoop:D_SMD_TH" (at 57.15 78.105 0)
+    (property "Footprint" "dumta:D_SMD_TH" (at 57.15 78.105 0)
       (effects (font (size 1.27 1.27)) hide)
     )
@@
       (effects (font (size 1.27 1.27)))
     )
-    (property "Footprint" "keyswitches:Kailh_socket_PG1350_reversible" (at 67.31 74.295 0)
+    (property "Footprint" "dumta:Kailh_socket_PG1350_reversible" (at 67.31 74.295 0)
       (effects (font (size 1.27 1.27)) hide)
     )
@@
       (effects (font (size 1.27 1.27)))
     )
-    (property "Footprint" "swoop:D_SMD_TH" (at 74.93 78.105 0)
+    (property "Footprint" "dumta:D_SMD_TH" (at 74.93 78.105 0)
       (effects (font (size 1.27 1.27)) hide)
     )
@@
       (effects (font (size 1.27 1.27)))
     )
-    (property "Footprint" "keyswitches:Kailh_socket_PG1350_reversible" (at 85.09 74.295 0)
+    (property "Footprint" "dumta:Kailh_socket_PG1350_reversible" (at 85.09 74.295 0)
       (effects (font (size 1.27 1.27)) hide)
     )
@@
       (effects (font (size 1.27 1.27)))
     )
-    (property "Footprint" "keyswitches:Kailh_socket_PG1350_reversible" (at 102.87 74.295 0)
+    (property "Footprint" "dumta:Kailh_socket_PG1350_reversible" (at 102.87 74.295 0)
       (effects (font (size 1.27 1.27)) hide)
     )
@@
       (effects (font (size 1.27 1.27)))
     )
-    (property "Footprint" "keyswitches:Kailh_socket_PG1350_reversible" (at 120.65 74.295 0)
+    (property "Footprint" "dumta:Kailh_socket_PG1350_reversible" (at 120.65 74.295 0)
       (effects (font (size 1.27 1.27)) hide)
     )
@@
       (effects (font (size 1.27 1.27)))
     )
-    (property "Footprint" "swoop:D_SMD_TH" (at 92.71 78.105 0)
+    (property "Footprint" "dumta:D_SMD_TH" (at 92.71 78.105 0)
       (effects (font (size 1.27 1.27)) hide)
     )
@@
       (effects (font (size 1.27 1.27)))
     )
-    (property "Footprint" "swoop:D_SMD_TH" (at 110.49 78.105 0)
+    (property "Footprint" "dumta:D_SMD_TH" (at 110.49 78.105 0)
       (effects (font (size 1.27 1.27)) hide)
     )
@@
       (effects (font (size 1.27 1.27)))
     )
-    (property "Footprint" "swoop:D_SMD_TH" (at 128.27 78.105 0)
+    (property "Footprint" "dumta:D_SMD_TH" (at 128.27 78.105 0)
       (effects (font (size 1.27 1.27)) hide)
     )
@@
       (effects (font (size 1.27 1.27)))
     )
-    (property "Footprint" "keyswitches:Kailh_socket_PG1350_reversible" (at 105.41 104.14 0)
+    (property "Footprint" "dumta:Kailh_socket_PG1350_reversible" (at 105.41 104.14 0)
       (effects (font (size 1.27 1.27)) hide)
     )
@@
       (effects (font (size 1.27 1.27)))
     )
-    (property "Footprint" "swoop:D_SMD_TH" (at 110.49 93.345 0)
+    (property "Footprint" "dumta:D_SMD_TH" (at 110.49 93.345 0)
       (effects (font (size 1.27 1.27)) hide)
     )
@@
       (effects (font (size 1.27 1.27)))
     )
-    (property "Footprint" "keyswitches:Kailh_socket_PG1350_reversible" (at 120.65 89.535 0)
+    (property "Footprint" "dumta:Kailh_socket_PG1350_reversible" (at 120.65 89.535 0)
       (effects (font (size 1.27 1.27)) hide)
     )
@@
       (effects (font (size 1.27 1.27)))
     )
-    (property "Footprint" "swoop:D_SMD_TH" (at 128.27 93.345 0)
+    (property "Footprint" "dumta:D_SMD_TH" (at 128.27 93.345 0)
       (effects (font (size 1.27 1.27)) hide)
     )
@@
       (effects (font (size 1.27 1.27)))
     )
-    (property "Footprint" "keyswitches:Kailh_socket_PG1350_reversible" (at 83.82 97.79 0)
+    (property "Footprint" "dumta:Kailh_socket_PG1350_reversible" (at 83.82 97.79 0)
       (effects (font (size 1.27 1.27)) hide)
     )
@@
       (effects (font (size 1.27 1.27)))
     )
-    (property "Footprint" "swoop:D_SMD_TH" (at 92.71 93.345 0)
+    (property "Footprint" "dumta:D_SMD_TH" (at 92.71 93.345 0)
       (effects (font (size 1.27 1.27)) hide)
     )
@@
       (effects (font (size 1.27 1.27)) (justify left))
     )
-    (property "Footprint" "swoop:Battery_pads_reversible" (at 137.16 115.316 90)
-      (effects (font (size 1.27 1.27)) hide)
-    )
+    (property "Footprint" "dumta:Battery_pads_reversible" (at 137.16 115.316 90)
+      (effects (font (size 1.27 1.27)) hide)
+    )
