File: hardware/pcb/temper.kicad_sch (KiCad schematic)
At the start: 41 parts, among them J2 nice_view, SW1 SW_PUSH, SW10 SW_PUSH, SW11 SW_PUSH, SW12 SW_PUSH, SW13 SW_PUSH, SW14 SW_PUSH, SW15 SW_PUSH, SW16 SW_PUSH, SW17 SW_PUSH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

Commit message: refactor: rename kicad project to temper, keeping the library name the same
Other:
- title: dumta -> temper
Changed lines of the file:
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@@
   (paper "A4")
   (title_block
-    (title "dumta")
-    (date "2023-07-07")
+    (title "temper")
+    (date "2023-07-14")
     (rev "1.0")
     (company "raeedcho")
